Commit message: urdf

File: Simulation/【装配体】自定义控制器（DM4310）/robot.urdf (robot description, URDF)
Before this commit: robot _装配体_自定义控制器_DM4310_, 8 links, 7 joints
Joints:
- joint joint2: origin xyz=7.170833143e-09 0.004000000024 -1.161850293e-12 rpy=1.570796326 1.047197552 -5.030947457e-10 -> xyz=7.170833143e-09 0.004000000024 -1.161850293e-12 rpy=1.570796327 0 0
- joint joint3: origin xyz=-4.316460807e-09 0.147999652 -4.090038924e-08 rpy=1.57079605 -0.04075675318 1.126955818e-08 -> xyz=-4.316460807e-09 0.147999652 -4.090038924e-08 rpy=1.570796327 0 0
- joint joint4: origin xyz=-2.838116055e-09 0.002502097331 4.376801019e-08 rpy=1.57083178 1.054802579 3.083716605e-05 -> xyz=-2.838116055e-09 0.002502097331 4.376801019e-08 rpy=1.570796327 0 0
- joint joint5: origin xyz=4.805759683e-07 -0.09999888857 2.365613278e-06 rpy=1.570772599 0.07758160177 -1.838953601e-06 -> xyz=4.805759683e-07 -0.09999888857 2.365613278e-06 rpy=1.570796327 0 0
- joint joint6: origin xyz=-8.497409919e-08 0.0009994027096 0 rpy=1.570796325 -1.546151804 2.670220361e-09 -> xyz=-8.497409919e-08 0.0009994027096 0 rpy=1.570796327 0 0
- joint joint7: origin xyz=1.312649219e-06 0 0 rpy=-1.570776404 1.216346404e-11 0 -> xyz=-1.312649219e-06 0 0 rpy=1.570796327 0 0
